File: pcb/microcontroller.kicad_sch (KiCad schematic)
At the start: 16 parts, among them J1 Conn_ARM_SWD_TagConnect_TC2030, J2 USB_C_Receptacle_USB2.0_14P, U2 STM32G431CBTx, U3 USBLC6-2SC6, Y1 8Mhz

Commit message: pcb: wip
Changed lines of the file:
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@@
 	)
 	(label "USB_D+"
-		(at 158.75 99.06 0)
+		(at 154.94 99.06 0)
 		(fields_autoplaced yes)
 		(effects
@@
 		(effects
 			(font
-				(size 1.27 1.27)
+				(size 1 1)
 				(bold yes)
 			)
@@
 		(effects
 			(font
-				(size 1.27 1.27)
+				(size 1 1)
 				(bold yes)
 			)
@@
 		(effects
 			(font
-				(size 1.27 1.27)
+				(size 1 1)
 				(bold yes)
 			)
@@
 		(effects
 			(font
-				(size 1.27 1.27)
+				(size 1 1)
 				(bold yes)
 			)
@@
 	)
 	(label "USB_D-"
-		(at 158.75 96.52 0)
+		(at 154.94 96.52 0)
 		(fields_autoplaced yes)
 		(effects

Commit message: pcb: first version schematic
Parts:
- removed J1: Conn_ARM_SWD_TagConnect_TC2030, Connector:Tag-Connect_TC2030-IDC-FP_2x03_P1.27mm_Vertical, symbol Connector:Conn_ARM_SWD_TagConnect_TC2030
- removed J2: USB_C_Receptacle_USB2.0_14P, symbol Connector:USB_C_Receptacle_USB2.0_14P
- removed R5: 220R, symbol Device:R
- added C29, C30, C31: 4n7, Capacitor_SMD:C_0603_1608Metric, symbol Device:C
- added R30, R31, R32: 10k, Resistor_SMD:R_0603_1608Metric, symbol Device:R
- added R33, R34, R35: 2k2, Resistor_SMD:R_0603_1608Metric, symbol Device:R
- C10, C11, C12, C7, C8, C9: footprint (none) -> Capacitor_SMD:C_0603_1608Metric
- D2: footprint (none) -> Diode_SMD:D_MiniMELF
- FB2, R6, R7: footprint (none) -> Resistor_SMD:R_0603_1608Metric
- Y1: value 8Mhz -> 24Mhz; footprint (none) -> tractions_symbols:better_crystal
Connections:
- net HSE is gone; now on net HSE_OUT: Y1.1
- net +5V: now also U3.5 (VBUS)
- net GND: now also C29.2, C30.2, C31.2
- net SWDIO: no longer U2.40 (PB3)
- net VDD: now also R33.2, R34.2, R35.2
- net VBUS: now reaches D2.2 (A)
- net VBUS: no longer U3.5 (VBUS)
- net SENS1: now reaches U2.10 (PA2)
- net VCC_SENSE: now reaches U2.14 (PA6)
- net BR_SO2: now reaches U2.16 (PB0)
- net BR_SO1: now reaches U2.17 (PB1)
- net FAULT: now reaches U2.2 (PC13)
- net UART_TX: now reaches U2.22 (PB10)
- net UART_RX: now reaches U2.25 (PB11)
- net USR_BUTTON: now reaches U2.26 (PB12)
- net L3: now reaches U2.27 (PB13)
- net L2: now reaches U2.28 (PB14)
- net L1: now reaches U2.29 (PB15)
- net OCTP: now reaches U2.3 (PC14)
- net H3: now reaches U2.30 (PA8)
- net H2: now reaches U2.31 (PA9)
- net H1: now reaches U2.32 (PA10)
- net EN: now reaches U2.39 (PA15)
- net DC_CAL: now reaches U2.4 (PC15)
- net at U2.42 (PB5): now also C29.1, R32.1, R33.1
- net at U2.43 (PB6): now also C30.1, R30.1, R34.1
- net at U2.44 (PB7): now also C31.1, R31.1, R35.1
- net SENS3: now reaches U2.8 (PA0)
- net SENS2: now reaches U2.9 (PA1)
- net CC1 renamed USBC_CC1
- net CC2 renamed USBC_CC2
- net SWD_NRST renamed SWD_RST
- new net HALL1_IN: R30.2
- new net HALL2_IN: R31.2
- new net HALL3_IN: R32.2
- new net SWO: U2.40 (PB3)
- no-connect marks 0 -> 8
Other:
- note added: "STM32G4"
- moved on the sheet: C10, C11, C12, C7, C8, C9, FB2, R6, R7, U2, U3, Y1

Commit message: pcb: v1.0 layout finsihed
Connections:
- net +5V: no longer U3.5 (VBUS)
- net GND: now also U3.5 (VBUS); no longer U3.2 (GND)
- net USBC_D+: now also U3.6 (I/O1); no longer U3.3 (I/O2)
- net USBC_D-: now also U3.4 (I/O2); no longer U3.1 (I/O1)
- net USB_D+: now also U3.1 (I/O1); no longer U3.4 (I/O2)
- net USB_D-: now also U3.3 (I/O2); no longer U3.6 (I/O1)
- net VBUS: now also U3.2 (GND)
Other:
- moved on the sheet: D2
Changed lines of the file:
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@@
 	)
 	(junction
-		(at 68.58 104.14)
+		(at 193.04 93.98)
 		(diameter 0)
 		(color 0 0 0 0)
 	)
 	(junction
-		(at 120.65 73.66)
+		(at 68.58 104.14)
 		(diameter 0)
 		(color 0 0 0 0)
 	)
 	(junction
-		(at 138.43 66.04)
+		(at 120.65 73.66)
 		(diameter 0)
 		(color 0 0 0 0)
 	)
 	(junction
-		(at 193.04 93.98)
+		(at 138.43 66.04)
 		(diameter 0)
 		(color 0 0 0 0)
@@
 	(wire
 		(pts
-			(xy 193.04 93.98) (xy 194.31 93.98)
-		)
-		(stroke
-			(width 0)
-			(type default)
-		)
-	)
-	(wire
-		(pts
 			(xy 120.65 137.16) (xy 123.19 137.16)
 		)
@@
 	(wire
 		(pts
-			(xy 193.04 109.22) (xy 193.04 111.76)
+			(xy 198.12 101.6) (xy 205.74 101.6)
 		)
 		(stroke
@@
 	(wire
 		(pts
-			(xy 193.04 90.17) (xy 193.04 93.98)
+			(xy 193.04 109.22) (xy 193.04 111.76)
 		)
 		(stroke
@@
 	(wire
 		(pts
-			(xy 120.65 91.44) (xy 123.19 91.44)
+			(xy 193.04 83.82) (xy 193.04 85.09)
 		)
 		(stroke
@@
 	(wire
 		(pts
-			(xy 140.97 147.32) (xy 140.97 149.86)
+			(xy 120.65 91.44) (xy 123.19 91.44)
 		)
 		(stroke
@@
 	(wire
 		(pts
-			(xy 86.36 119.38) (xy 99.06 119.38)
+			(xy 140.97 147.32) (xy 140.97 149.86)
 		)
 		(stroke
@@
 	(wire
 		(pts
-			(xy 198.12 101.6) (xy 204.47 101.6)
+			(xy 86.36 119.38) (xy 99.06 119.38)
 		)
 		(stroke
@@
 	(wire
 		(pts
-			(xy 193.04 96.52) (xy 193.04 93.98)
-		)
-		(stroke
-			(width 0)
-			(type default)
-		)
-	)
-	(wire
-		(pts
 			(xy 80.01 114.3) (xy 80.01 123.19)
 		)
@@
 	(wire
 		(pts
+			(xy 193.04 93.98) (xy 193.04 96.52)
+		)
+		(stroke
+			(width 0)
+			(type default)
+		)
+	)
+	(wire
+		(pts
+			(xy 193.04 93.98) (xy 196.85 93.98)
+		)
+		(stroke
+			(width 0)
+			(type default)
+		)
+	)
+	(wire
+		(pts
 			(xy 100.33 46.99) (xy 113.03 46.99)
 		)
@@
 	(wire
 		(pts
+			(xy 198.12 104.14) (xy 205.74 104.14)
+		)
+		(stroke
+			(width 0)
+			(type default)
+		)
+	)
+	(wire
+		(pts
 			(xy 100.33 49.53) (xy 100.33 46.99)
 		)
@@
 	(wire
 		(pts
+			(xy 193.04 92.71) (xy 193.04 93.98)
+		)
+		(stroke
+			(width 0)
+			(type default)
+		)
+	)
+	(wire
+		(pts
 			(xy 77.47 116.84) (xy 88.9 116.84)
 		)
@@
 	(wire
 		(pts
-			(xy 198.12 104.14) (xy 204.47 104.14)
-		)
-		(stroke
-			(width 0)
-			(type default)
-		)
-	)
-	(wire
-		(pts
 			(xy 219.71 109.22) (xy 227.33 109.22)
 		)
@@
 	)
 	(label "USBC_D+"
-		(at 199.39 104.14 0)
+		(at 201.93 104.14 0)
 		(fields_autoplaced yes)
 		(effects
@@
 	)
 	(label "USBC_D-"
-		(at 199.39 101.6 0)
+		(at 201.93 101.6 0)
 		(fields_autoplaced yes)
 		(effects
@@
 	(hierarchical_label "USBC_D+"
 		(shape bidirectional)
-		(at 204.47 104.14 0)
+		(at 205.74 104.14 0)
 		(fields_autoplaced yes)
 		(effects
@@
 	(hierarchical_label "USBC_D-"
 		(shape bidirectional)
-		(at 204.47 101.6 0)
+		(at 205.74 101.6 0)
 		(fields_autoplaced yes)
 		(effects
@@
 	(hierarchical_label "VBUS"
 		(shape input)
-		(at 201.93 93.98 0)
+		(at 196.85 93.98 0)
 		(fields_autoplaced yes)
 		(effects
@@
 	(symbol
 		(lib_id "Power_Protection:USBLC6-2SC6")
-		(at 193.04 101.6 0)
-		(mirror y)
+		(at 193.04 104.14 0)
+		(mirror x)
 		(unit 1)
 		(exclude_from_sim no)
@@
 		(fields_autoplaced yes)
 		(property "Reference" "U3"
-			(at 191.3889 93.98 0)
+			(at 194.6911 111.76 0)
 			(effects
 				(font
@@
 		)
 		(property "Value" "USBLC6-2SC6"
-			(at 191.3889 96.52 0)
+			(at 194.6911 109.22 0)
 			(effects
 				(font
@@
 		)
 		(property "Footprint" "Package_TO_SOT_SMD:SOT-23-6"
-			(at 191.77 107.95 0)
+			(at 194.31 97.79 0)
 			(effects
 				(font
@@
 		)
 		(property "Datasheet" "https://www.st.com/resource/en/datasheet/usblc6-2.pdf"
-			(at 191.77 109.855 0)
+			(at 194.31 95.885 0)
 			(effects
 				(font
@@
 		)
 		(property "Description" "Very low capacitance ESD protection diode, 2 data-line, SOT-23-6"
-			(at 193.04 101.6 0)
+			(at 193.04 104.14 0)
 			(effects
 				(font
@@
 	(symbol
 		(lib_id "power:+5V")
-		(at 193.04 90.17 0)
+		(at 193.04 83.82 0)
 		(unit 1)
 		(exclude_from_sim no)
@@
 		(fields_autoplaced yes)
 		(property "Reference" "#PWR020"
-			(at 193.04 93.98 0)
+			(at 193.04 87.63 0)
 			(effects
 				(font
@@
 		)
 		(property "Value" "+5V"
-			(at 193.04 85.09 0)
+			(at 193.04 78.74 0)
 			(effects
 				(font
@@
 		)
 		(property "Footprint" ""
-			(at 193.04 90.17 0)
+			(at 193.04 83.82 0)
 			(effects
 				(font
@@
 		)
 		(property "Datasheet" ""
-			(at 193.04 90.17 0)
+			(at 193.04 83.82 0)
 			(effects
 				(font
@@
 		)
 		(property "Description" "Power symbol creates a global label with name \"+5V\""
-			(at 193.04 90.17 0)
+			(at 193.04 83.82 0)
 			(effects
 				(font
@@
 		(on_board yes)
 		(dnp no)
-		(fields_autoplaced yes)
 		(property "Reference" "#PWR018"
 			(at 193.04 118.11 0)
@@
 		)
 		(property "Value" "GND"
-			(at 193.04 116.84 0)
+			(at 210.82 97.79 0)
 			(effects
 				(font
@@
 	(symbol
 		(lib_id "Device:D")
-		(at 198.12 93.98 0)
+		(at 193.04 88.9 270)
 		(unit 1)
 		(exclude_from_sim no)
@@
 		(fields_autoplaced yes)
 		(property "Reference" "D2"
-			(at 198.12 87.63 0)
+			(at 195.58 87.6299 90)
 			(effects
 				(font
 					(size 1.27 1.27)
 				)
+				(justify left)
 			)
 		)
 		(property "Value" "D"
-			(at 198.12 90.17 0)
+			(at 195.58 90.1699 90)
 			(effects
 				(font
 					(size 1.27 1.27)
 				)
+				(justify left)
 			)
 		)
 		(property "Footprint" "Diode_SMD:D_MiniMELF"
-			(at 198.12 93.98 0)
+			(at 193.04 88.9 0)
 			(effects
 				(font
@@
 		)
 		(property "Datasheet" "~"
-			(at 198.12 93.98 0)
+			(at 193.04 88.9 0)
 			(effects
 				(font
@@
 		)
 		(property "Description" "Diode"
-			(at 198.12 93.98 0)
+			(at 193.04 88.9 0)
 			(effects
 				(font
@@
 		)
 		(property "Sim.Device" "D"
-			(at 198.12 93.98 0)
+			(at 193.04 88.9 0)
 			(effects
 				(font
@@
 		)
 		(property "Sim.Pins" "1=K 2=A"
-			(at 198.12 93.98 0)
+			(at 193.04 88.9 0)
 			(effects
 				(font
